Commit message: Added needed configurations and stls for rbsherpa_xl

File: rbsherpa_description/robots/rbsherpa_xl.urdf.xacro (robot description, xacro)
@@ -17,11 +17,11 @@
     <xacro:property name="deg2rad" value="0.01745329251"/>
     <!-- Wheel parameters -->
-    <xacro:property name="wheel_offset_x" value="0.4655" />    <!-- x,y,z in translation from base_link to the center of the wheel -->
-    <xacro:property name="wheel_offset_y" value="0.294" />
+    <xacro:property name="wheel_offset_x" value="0.4795" />    <!-- x,y,z in translation from base_link to the center of the wheel -->
+    <xacro:property name="wheel_offset_y" value="0.2925" />
     <xacro:property name="wheel_offset_z" value="0.0" />
-    <!-- Wheel parameters -->
-    <xacro:property name="G2_offset_x" value="0.17286" />
+    <!-- Bi-arm support parameters -->
+    <xacro:property name="G2_offset_x" value="0.207" />
     <xacro:property name="G2_offset_y" value="0.0" />
-    <xacro:property name="G2_offset_z" value="0.50288" />
+    <xacro:property name="G2_offset_z" value="0.57188" />
     <!-- Flag to select the high or low quality model -->
     <xacro:property name="hq" value="true" />
@@ -57,5 +57,5 @@
         <!-- IMU -->
         <!--xacro:sensor_imu_hector prefix="${prefix}imu" parent="${prefix}base_link">
-            <origin xyz="0.3 0.3 0.250" rpy="0 0 0"/>
+            <origin xyz="0.3 0.0 0.3" rpy="0 0 0"/>
         </xacro:sensor_imu_hector-->
         <!-- GPS -->

File: rbsherpa_description/urdf/bases/bi_arm_support.urdf.xacro (robot description, xacro)
@@ -1,5 +1,5 @@
 <?xml version="1.0"?>
 <robot xmlns:xacro="http://wiki.ros.org/xacro">
-	<xacro:include filename="$(find ur_description)/urdf/ur10.urdf.xacro" />
+	<xacro:include filename="$(find ur_e_description)/urdf/ur10e.urdf.xacro" />
   <xacro:include filename="$(find rbsherpa_description)/urdf/inertia.urdf.xacro" />
   <xacro:property name="M_PI" value="3.1415926535897931" />
@@ -13,7 +13,7 @@
     <link name="${prefix}G2_link">
       <visual>
-        <origin xyz="0 0 0" rpy="0 0 ${M_PI/2.0}" />
+        <origin xyz="0.0 0.0 0.0" rpy="0 0 ${M_PI/2.0}" />
         <geometry>
-          <mesh filename="package://rbsherpa_description/meshes/bases/bi_arm_support.stl" />
+          <mesh filename="package://rbsherpa_description/meshes/bases/bi_arm_support_rbsherpa_xl.stl" />
         </geometry>
       </visual>
@@ -21,10 +21,10 @@
         <origin xyz="0 0 0" rpy="0 0 ${M_PI/2.0}" />
         <geometry>
-          <mesh filename="package://rbsherpa_description/meshes/bases/bi_arm_support.stl" />
+          <mesh filename="package://rbsherpa_description/meshes/bases/bi_arm_support_rbsherpa_xl.stl" />
         </geometry>
       </collision>
       <inertial>
-        <mass value="10" />
-        <origin xyz="0 0 0" rpy="${M_PI/2.0} 0 0"/>
+        <mass value="5" />
+        <origin xyz="0 0 0" rpy="0 0 ${M_PI/2.0}"/>
         <solid_cuboid_inertia  w="0.4" h="0.4" d="0.2" m="5"/>
       </inertial>
@@ -43,48 +43,48 @@
     <xacro:if value="${load_kinematics_file}">
       <joint name="${prefix}left_arm_base_joint" type="fixed">
-        <origin xyz="0 0.13861 0.10943" rpy="0.902 0 3.1416"/>
+        <origin xyz="0 0.0915 0.15044" rpy="0.9 0 3.1416"/>
         <parent link="${prefix}G2_link" />
         <child link="${prefix}left_arm_base_link" />
       </joint>
-      <xacro:ur10_robot prefix="${prefix}left_arm_" joint_limited="true"
+      <xacro:ur10e_robot prefix="${prefix}left_arm_" joint_limited="true"
         shoulder_pan_lower_limit="${-pi}" shoulder_pan_upper_limit="${pi}"
         wrist_3_lower_limit="${-pi}" wrist_3_upper_limit="${pi}"
-        kinematics_file="${load_yaml('$(find rbsherpa_control)/config/calibration/ur10_calibration.yaml')}">
-      </xacro:ur10_robot>
+        kinematics_file="${load_yaml('$(find rbsherpa_control)/config/calibration/ur10e_default.yaml')}">
+      </xacro:ur10e_robot>
     </xacro:if>
     <xacro:unless value="${load_kinematics_file}">
       <joint name="${prefix}left_arm_base_joint" type="fixed">
-        <origin xyz="0 0.13861 0.10943" rpy="0.902 0 3.1416"/>
+        <origin xyz="0 -0.0915 0.15044" rpy="0.9 0 3.1416"/>
         <parent link="${prefix}G2_link" />
         <child link="${prefix}right_arm_base_link" />
       </joint>
-      <xacro:ur10_robot prefix="${prefix}left_arm_" joint_limited="true"
+      <xacro:ur10e_robot prefix="${prefix}left_arm_" joint_limited="true"
         shoulder_pan_lower_limit="${-pi}" shoulder_pan_upper_limit="${pi}"
         wrist_3_lower_limit="${-pi}" wrist_3_upper_limit="${pi}">
-      </xacro:ur10_robot>
+      </xacro:ur10e_robot>
     </xacro:unless>
     <!-- Right UR10 -->
     <xacro:if value="${load_kinematics_file}">
       <joint name="${prefix}right_arm_base_joint" type="fixed">
-        <origin xyz="0 -0.13861 0.10943" rpy="0.902 0 0"/>
+        <origin xyz="0 -0.0915 0.15044" rpy="0.9 0 0"/>
         <parent link="${prefix}G2_link" />
         <child link="${prefix}right_arm_base_link" />
       </joint>
-      <xacro:ur10_robot prefix="${prefix}right_arm_" joint_limited="true"
+      <xacro:ur10e_robot prefix="${prefix}right_arm_" joint_limited="true"
         shoulder_pan_lower_limit="${-pi}" shoulder_pan_upper_limit="${pi}"
         wrist_3_lower_limit="${-pi}" wrist_3_upper_limit="${pi}"
-        kinematics_file="${load_yaml('$(find rbsherpa_control)/config/calibration/ur10_calibration.yaml')}">
-      </xacro:ur10_robot>
+        kinematics_file="${load_yaml('$(find rbsherpa_control)/config/calibration/ur10e_default.yaml')}">
+      </xacro:ur10e_robot>
     </xacro:if>
     <xacro:unless value="${load_kinematics_file}">
       <joint name="${prefix}right_arm_base_joint" type="fixed">
-        <origin xyz="0 -0.13861 0.10943" rpy="0.902 0 0"/>
+        <origin xyz="0 -0.0915 0.15044" rpy="0.9 0 0"/>
         <parent link="${prefix}G2_link" />
         <child link="${prefix}right_arm_base_link" />
       </joint>
-      <xacro:ur10_robot prefix="${prefix}right_arm_" joint_limited="true"
+      <xacro:ur10e_robot prefix="${prefix}right_arm_" joint_limited="true"
         shoulder_pan_lower_limit="${-pi}" shoulder_pan_upper_limit="${pi}"
         wrist_3_lower_limit="${-pi}" wrist_3_upper_limit="${pi}">
-      </xacro:ur10_robot>
+      </xacro:ur10e_robot>
     </xacro:unless>
   </xacro:macro>

File: rbsherpa_description/urdf/bases/rbsherpa_xl_base.urdf.xacro (robot description, xacro)
@@ -25,10 +25,10 @@
     </xacro:if>
     <!-- BASE_LINK -->
-    <link name="${prefix}base_link">   x:1.025 y:0.75 z:0.3
+    <link name="${prefix}base_link">
       <inertial>
         <mass value="25.0" />
-        <origin xyz="0 0 0.35" />
+        <origin xyz="0 0 0.376" />
         <!--inertia ixx="1.0" ixy="0.0" ixz="0.0" iyy="1.0" iyz="0.0" izz="1.0" /-->
-        <solid_cuboid_inertia  w="1.025" h="0.75" d="0.3" m="25"/>
+        <solid_cuboid_inertia  w="1.265" h="0.812" d="0.465" m="25"/>
       </inertial>
       <visual>
@@ -36,10 +36,10 @@
         <xacro:if value="${hq}">
           <geometry>
-            <mesh filename="package://rbsherpa_description/meshes/bases/rbsherpa_xl_chassis.stl"/>
+            <mesh filename="package://rbsherpa_description/meshes/bases/rbsherpa_xl_base.stl"/>
           </geometry>
         </xacro:if>
         <xacro:unless value="${hq}">
           <geometry>
-            <mesh filename="package://rbsherpa_description/meshes/bases/rbsherpa_xl_chassis.stl"/>
+            <mesh filename="package://rbsherpa_description/meshes/bases/rbsherpa_xl_base.stl"/>
           </geometry>
         </xacro:unless>
@@ -51,5 +51,5 @@
         <origin xyz="0 0 0" rpy="0 0 0 " />
         <geometry>
-          <mesh filename="package://rbsherpa_description/meshes/bases/rbsherpa_xl_chassis.stl"/>
+          <mesh filename="package://rbsherpa_description/meshes/bases/rbsherpa_xl_base.stl"/>
         </geometry>
       </collision>

File: rbsherpa_description/urdf/wheels/motor_wheel_xl.urdf.xacro (robot description, xacro)
@@ -3,7 +3,7 @@
   <xacro:property name="M_PI" value="3.1415926535897931" />
   <!-- Wheels -->
-  <xacro:property name="wheel_radius" value="0.170" />
-  <xacro:property name="wheel_height" value="0.170" />
-  <xacro:property name="wheel_mass" value="5.0" />
+  <xacro:property name="wheel_radius" value="0.17" />
+  <xacro:property name="wheel_width" value="0.14" />
+  <xacro:property name="wheel_mass" value="4.0" />
   <!-- in kg-->
   <xacro:property name="steer_joint_damping" value="2.0" />
@@ -46,11 +46,11 @@
         <!-- HIGH RESOLUTION WHEELS -->
         <xacro:if value="${hq}">
-          <origin xyz="0 0 0.205" rpy="0 0 3.1416" />
+          <origin xyz="0 0 0.27952" rpy="0 0 0" />
           <geometry>
             <xacro:if value="${reflect}">
-              <mesh filename="package://rbsherpa_description/meshes/wheels/L.stl" />
+              <mesh filename="package://rbsherpa_description/meshes/wheels/hub_rbsherpa_xl.stl" />
             </xacro:if>
             <xacro:unless value="${reflect}">
-              <mesh filename="package://rbsherpa_description/meshes/wheels/L.stl" />
+              <mesh filename="package://rbsherpa_description/meshes/wheels/hub_rbsherpa_xl.stl" />
             </xacro:unless>
           </geometry>
@@ -58,11 +58,11 @@
         <!-- LOW RESOLUTION WHEELS -->
         <xacro:unless value="${hq}">
-          <origin xyz="0 0 0.205" rpy="0 0 3.1416" />
+          <origin xyz="0 0 0.27952" rpy="0 0 0" />
           <geometry>
             <xacro:if value="${reflect}">
-              <mesh filename="package://rbsherpa_description/meshes/wheels/L.stl" />
+              <mesh filename="package://rbsherpa_description/meshes/wheels/hub_rbsherpa_xl.dae" />
             </xacro:if>
             <xacro:unless value="${reflect}">
-              <mesh filename="package://rbsherpa_description/meshes/wheels/L.stl" />
+              <mesh filename="package://rbsherpa_description/meshes/wheels/hub_rbsherpa_xl.dae" />
             </xacro:unless>
           </geometry>
@@ -70,18 +70,19 @@
       </visual>
       <collision>
-        <origin xyz="0 0 0.205" rpy="0 0 3.1416" />
+        <origin xyz="0 0 0.27952" rpy="0 0 0" />
         <geometry>
           <xacro:if value="${reflect}">
-            <mesh filename="package://rbsherpa_description/meshes/wheels/L.stl" />
+            <mesh filename="package://rbsherpa_description/meshes/wheels/hub_rbsherpa_xl.dae" />
           </xacro:if>
           <xacro:unless value="${reflect}">
-            <mesh filename="package://rbsherpa_description/meshes/wheels/L.stl" />
+            <mesh filename="package://rbsherpa_description/meshes/wheels/hub_rbsherpa_xl.dae" />
           </xacro:unless>
         </geometry>
       </collision>
       <inertial>
-        <mass value="10" />
-        <origin xyz="0 0 0" />
-        <inertia ixx="0.01" ixy="0.0" ixz="0.0" iyy="0.01" iyz="0.0" izz="0.01" />
+        <mass value="4" />
+        <origin xyz="0 0 0.12" rpy="0 0 0"/>
+        <!--inertia ixx="0.01" ixy="0.0" ixz="0.0" iyy="0.01" iyz="0.0" izz="0.01" /-->
+        <cylinder_inertia m="${wheel_mass}" r="${wheel_radius}" h="${wheel_width}" />
       </inertial>
     </link>
@@ -122,8 +123,8 @@
           <geometry>
             <xacro:if value="${reflect}">
-              <mesh filename="package://rbsherpa_description/meshes/wheels/wheel_xl.stl" />
+              <mesh filename="package://rbsherpa_description/meshes/wheels/wheel_rbsherpa_xl.stl" />
             </xacro:if>
             <xacro:unless value="${reflect}">
-              <mesh filename="package://rbsherpa_description/meshes/wheels/wheel_xl.stl" />
+              <mesh filename="package://rbsherpa_description/meshes/wheels/wheel_rbsherpa_xl.stl" />
             </xacro:unless>
           </geometry>
@@ -134,8 +135,8 @@
           <geometry>
             <xacro:if value="${reflect}">
-              <mesh filename="package://rbsherpa_description/meshes/wheels/wheel_xl.dae" />
+              <mesh filename="package://rbsherpa_description/meshes/wheels/wheel_rbsherpa_xl.dae" />
             </xacro:if>
             <xacro:unless value="${reflect}">
-              <mesh filename="package://rbsherpa_description/meshes/wheels/wheel_xl.dae" />
+              <mesh filename="package://rbsherpa_description/meshes/wheels/wheel_rbsherpa_xl.dae" />
             </xacro:unless>
           </geometry>
@@ -146,8 +147,8 @@
         <geometry>
           <xacro:if value="${reflect}">
-            <mesh filename="package://rbsherpa_description/meshes/wheels/wheel_xl.stl" />
+            <mesh filename="package://rbsherpa_description/meshes/wheels/collision_wheel_rbsherpa_xl.dae" />
           </xacro:if>
           <xacro:unless value="${reflect}">
-            <mesh filename="package://rbsherpa_description/meshes/wheels/wheel_xl.stl" />
+            <mesh filename="package://rbsherpa_description/meshes/wheels/collision_wheel_rbsherpa_xl.dae" />
           </xacro:unless>
         </geometry>
@@ -156,5 +157,5 @@
         <mass value="${wheel_mass}" />
         <origin xyz="0 0 0" rpy="${M_PI/2} 0 0"/>
-        <cylinder_inertia m="${wheel_mass}" r="${wheel_radius}" h="${wheel_height}" />
+        <cylinder_inertia m="${wheel_mass}" r="${wheel_radius}" h="${wheel_width}" />
       </inertial>
     </link>

Commit message: Updated config for UR10e

File: rbsherpa_description/robots/rbsherpa_xl.urdf.xacro (robot description, xacro)
@@ -56,11 +56,15 @@
         <!-- SENSORS see robotnik_sensors for the specific configuration -->
         <!-- IMU -->
-        <!--xacro:sensor_imu_hector prefix="${prefix}imu" parent="${prefix}base_link">
+        <xacro:sensor_imu_hector prefix="${prefix}imu" parent="${prefix}base_link">
             <origin xyz="0.3 0.0 0.3" rpy="0 0 0"/>
-        </xacro:sensor_imu_hector-->
+        </xacro:sensor_imu_hector>
         <!-- GPS -->
         <!--xacro:sensor_gps prefix="${prefix}gps" parent="${prefix}base_link">
-            <origin xyz="-0.04625 0.0 1.115" rpy="0 0 0"/>
+            <origin xyz="-0.04625 0.0 0.59188" rpy="0 0 0"/>
         </xacro:sensor_gps-->
+        <!-- Lidar -->
+        <!--xacro:sensor_rslidar_16 prefix="${prefix}front_ss_laser" parent="${prefix}base_link" gpu="true">
+            <origin xyz="0.511 0 0.21" rpy="0 0 0"/>
+        </xacro:sensor_rslidar_16-->
         <!-- Solid-State laser -->
         <!--xacro:sensor_benewake_ce30c prefix="${prefix}front_ss_laser" parent="${prefix}base_link" gpu="false">
